File: PCB/EE327 KiCAD Files/EE327 - Battery Management/EE327 - Battery Management.kicad_sch (KiCad schematic)
At the start: 0 parts

Commit message: Created Power Management Schematic Draft
Parts:
- added BT1: Battery, symbol Device:Battery
- added C1: 1u, symbol Device:C
- added C10, C11, C3, C4: 100n, symbol Device:C
- added C12: 2.2u, symbol Device:C
- added C13: 80u, symbol Device:C
- added C2: 100n, symbol Device:C_Polarized_US
- added C5: 470n, symbol Device:C
- added C6, C7, C8, C9: 4.7u, symbol Device:C
- added D1: D_Zener, symbol Device:D_Zener
- added D2, D3: D, symbol Device:D
- added L1: 47u, symbol Device:L
- added Q1, Q2, Q3, Q4, Q5, Q6, Q7, Q8: 2N7000, Package_TO_SOT_THT:TO-92_Inline, symbol Transistor_FET:2N7000
- added R1, R17: 220k, symbol Device:R
- added R10, R11, R12, R13, R14, R15, R16, R9: 10k, symbol Device:R
- added R18: 82k, symbol Device:R
- added R19, R20, R7, R8: 10, symbol Device:R
- added R2: 12k, symbol Device:R
- added R21: 2m, symbol Device:R
- added R22: 2, symbol Device:R
- added R3: 3k, symbol Device:R
- added R4: 75k, symbol Device:R
- added R5: 100k, symbol Device:R
- added R6: 5m, symbol Device:R
- added U1: BQ25751RRVR, VQFN36_RRV_TEX, symbol BQ25751RRVR:BQ25751RRVR
Connections:
- new net: D1.2 (A), Q5.1 (S), Q6.1 (S)
- new net: Q6.3 (D), R19.1, R21.1
- new net: R17.1, U1.9 (ICHG)
- new net: C12.1, R22.2
- new net: Q8.3 (D), R6.1, R7.2
- new net: R18.1, U1.10 (ILIM_HIZ)
- new net *INT: R12.2, U1.3 (*INT)
- new net *PG: R9.2, U1.6 (*PG)
- new net 12VDC: C1.1, Q5.3 (D), R2.1, U1.33 (VAC), U1.34 (ACUV)
- new net ACDRV: D1.1 (K), Q5.2 (G), Q6.2 (G), U1.31 (ACDRV)
- new net ACN: C11.2, R20.2, U1.29 (ACN)
- new net ACOV: R2.2, R3.1, U1.35 (ACOV)
- new net ACP: C10.1, R19.2, U1.30 (ACP)
- new net BATDRV: Q7.2 (G), Q8.2 (G), U1.15 (BATDRV)
- new net BATSRC: Q7.1 (S), Q8.1 (S), U1.16 (BATSRC)
- new net BTSD1: U1.26 (BTST1)
- new net BTSD2: U1.20 (BTST2)
- new net BTST1: C8.2, D2.1 (K)
- new net BTST2: C9.2, D3.1 (K)
- new net FB: R1.2, R4.1, U1.12 (FB)
- new net FBG: R4.2, U1.11 (FBG)
- new net FSW: R5.1, U1.36 (FSW_SYNC)
- new net GND: BT1.2 (-), C1.2, C10.2, C11.1, C12.2, C13.2, C3.2, C4.1, C6.2, C7.2, Q2.1 (S), Q4.1 (S), R16.2, R17.2, R18.2, R3.2, R5.2, U1.17 (MODE), U1.22 (PGND), U1.37 (PGND), U1.7 (*CE)
- new net HIDRV1: Q1.2 (G), U1.27 (HIDRV1)
- new net HIDRV2: Q3.2 (G), U1.19 (HIDRV2)
- new net LODRV1: Q2.2 (G), U1.25 (LODRV1)
- new net LODRV2: Q4.2 (G), U1.21 (LODRV2)
- new net REGN: C6.1, C7.1, D2.2 (A), D3.2 (A), R15.1, U1.23 (DRV_SUP), U1.24 (REGN)
- new net SCL: R14.2, U1.1 (SCL)
- new net SDA: R13.2, U1.2 (SDA)
- new net SRN: C4.2, C5.2, R8.1, U1.13 (SRN)
- new net SRP: C3.1, C5.1, R7.1, U1.14 (SRP)
- new net STAT1: R11.2, U1.4 (STAT1)
- new net STAT2: R10.2, U1.5 (STAT2)
- new net SW1: C8.1, L1.1, Q1.1 (S), Q2.3 (D), U1.28 (SW1)
- new net SW2: C9.1, L1.2, Q3.1 (S), Q4.3 (D), U1.18 (SW2)
- new net SYS: C13.1, C2.1, Q1.3 (D), Q3.3 (D), Q7.3 (D), R20.1, R21.2, R22.1, U1.32 (SYS)
- new net TS: R15.2, R16.1, U1.8 (TS)
- new net VESP: R10.1, R11.1, R12.1, R13.1, R14.1, R9.1
- new net Vbat: BT1.1 (+), R1.1, R6.2, R8.2
Other:
- note added: "Does not need to be made during test (Could be good indicator though...)"
- note added: "Open circuit for first tests"
- note added: "R1 = 0"
- note added: "Short for first tests"
- note added: "Transistor Part Numbers might be changed"
