File: PCB/EE327 KiCAD Files/EE327 - Battery Management/EE327 - Battery Management.kicad_sch (KiCad schematic)
At the start: 50 parts, among them Q1 2N7000, Q2 2N7000, Q3 2N7000, Q4 2N7000, Q5 2N7000, Q6 2N7000, Q7 2N7000, Q8 2N7000, U1 BQ25751RRVR

Commit message: Final PMIC Schematic
Parts:
- removed C10, C11: 100n, symbol Device:C
- removed C6: 4.7u, symbol Device:C
- removed R19, R20: 10, symbol Device:R
- removed R21: 2m, symbol Device:R
- L1: value 47u -> 10u
- R17: value 220k -> 920
- R6: value 5m -> 1
Connections:
- net ACP is gone; now on net ACN: U1.30 (ACP)
- net SYS is gone; now on net ACN: C13.1, C2.1, Q1.3 (D), Q7.3 (D), R22.1, U1.32 (SYS)
- net ACN: now also Q6.3 (D)
- net REGN: now also C7.1, R15.1, U1.23 (DRV_SUP), U1.24 (REGN)
- net VESP: no longer R15.1, U1.23 (DRV_SUP)
