File: PCB/EE327 KiCAD Files/EE327 - Battery Management (Schematic Only)/EE327 - Battery Management.kicad_sch (KiCad schematic)
At the start: 49 parts, among them Q1 2N7000, Q2 2N7000, Q3 2N7000, Q4 2N7000, Q5 2N7000, Q6 2N7000, Q7 2N7000, Q8 2N7000, U1 BQ25751RRVR

Commit message: Final Schematic Version
Parts:
- removed C10, C11: 100n, symbol Device:C
- removed C7: 4.7u, symbol Device:C
- removed R19, R20: 10, symbol Device:R
- removed R21: 2m, symbol Device:R
- L1: value 47u -> 10u
- Q1, Q2, Q3, Q4, Q5, Q6, Q7, Q8: value 2N7000 -> IRL520N
- R10, R11, R12, R13, R14, R15, R16, R9: value 10k -> 12k
- R17: value 220k -> 920
- R6: value 5m -> 1
Connections:
- net ACP is gone; now on net ACN: U1.30 (ACP)
- net ACN: now also C13.1, C2.1, Q1.3 (D), Q6.3 (D), Q7.3 (D), R22.1, U1.32 (SYS)
- net at Q8.3 (D), R6.1, R7.2: now also Q3.3 (D)
- net 12VDC renamed 5VDC
- removed net SYS: C13.1, C2.1, Q1.3 (D), Q3.3 (D), Q7.3 (D), R22.1, U1.32 (SYS)
Other:
- note removed: "Does not need to be made during test (Could be good indicator though...)"
- note removed: "Open circuit for first tests"
- note removed: "Short for first tests"
- note removed: "Transistor Part Numbers might be changed"
